Commit message: feat: baseline stable Ignition simulation with 4WD skid-steer, LiDAR/IMU, and indoor maze

File: src/outdoor_sim/urdf/robot_sensors.xacro (robot description, xacro)
@@ -1,89 +1,91 @@
 <?xml version="1.0"?>
 <robot xmlns:xacro="http://www.ros.org/wiki/xacro" name="outdoor_bot">
-  <!-- ============================================================ -->
-  <!-- 基础常量                                                       -->
-  <!-- ============================================================ -->
   <xacro:property name="M_PI" value="3.1415926535897931" />
-  <!-- ============================================================ -->
-  <!-- Base Link —— 机器人底盘                                        -->
-  <!-- ============================================================ -->
-  <link name="base_link">
+  <!-- Base Link —— 底盘 -->
+  <link name="body">
     <visual>
-      <geometry>
-        <box size="0.4 0.3 0.15"/>
-      </geometry>
-      <material name="blue">
-        <color rgba="0 0 0.8 1"/>
-      </material>
+      <geometry><box size="0.4 0.3 0.15"/></geometry>
+      <material name="blue"><color rgba="0 0 0.8 1"/></material>
     </visual>
     <collision>
-      <geometry>
-        <box size="0.4 0.3 0.15"/>
-      </geometry>
+      <geometry><box size="0.4 0.3 0.15"/></geometry>
     </collision>
     <inertial>
       <mass value="10.0"/>
-      <inertia ixx="0.09" ixy="0.0" ixz="0.0"
-               iyy="0.15" iyz="0.0"
-               izz="0.2"/>
+      <inertia ixx="0.09" ixy="0.0" ixz="0.0" iyy="0.15" iyz="0.0" izz="0.2"/>
     </inertial>
   </link>
   <!-- ============================================================ -->
-  <!-- LiDAR Link —— 物理实体                                        -->
+  <!-- 4WD 轮子定义与关节 (4x Wheels & Continuous Joints)             -->
+  <!-- ============================================================ -->
+  <xacro:macro name="wheel" params="prefix x_reflect y_reflect">
+    <link name="${prefix}_wheel">
+      <visual>
+        <origin xyz="0 0 0" rpy="${M_PI/2} 0 0"/>
+        <geometry><cylinder radius="0.08" length="0.04"/></geometry>
+        <material name="black"><color rgba="0 0 0 1"/></material>
+      </visual>
+      <collision>
+        <origin xyz="0 0 0" rpy="${M_PI/2} 0 0"/>
+        <geometry><cylinder radius="0.08" length="0.04"/></geometry>
+      </collision>
+      <inertial>
+        <mass value="0.5"/>
+        <inertia ixx="0.001" ixy="0.0" ixz="0.0" iyy="0.001" iyz="0.0" izz="0.001"/>
+      </inertial>
+    </link>
+    <joint name="${prefix}_wheel_joint" type="continuous">
+      <parent link="body"/>
+      <child link="${prefix}_wheel"/>
+      <!-- 轮子质心略低于底盘，使其能触地 -->
+      <origin xyz="${x_reflect*0.15} ${y_reflect*0.18} -0.05" rpy="0 0 0"/>
+      <axis xyz="0 1 0"/>
+    </joint>
+  </xacro:macro>
+  <xacro:wheel prefix="left_front" x_reflect="1" y_reflect="1" />
+  <xacro:wheel prefix="right_front" x_reflect="1" y_reflect="-1" />
+  <xacro:wheel prefix="left_rear" x_reflect="-1" y_reflect="1" />
+  <xacro:wheel prefix="right_rear" x_reflect="-1" y_reflect="-1" />
+  <!-- ============================================================ -->
+  <!-- 传感器 Link 保持不变                                          -->
   <!-- ============================================================ -->
   <link name="lidar_link">
     <visual>
       <origin xyz="0 0 0" rpy="0 0 0"/>
-      <geometry>
-        <cylinder radius="0.05" length="0.05"/>
-      </geometry>
-      <material name="black">
-        <color rgba="0 0 0 1"/>
-      </material>
+      <geometry><cylinder radius="0.05" length="0.05"/></geometry>
+      <material name="black"><color rgba="0 0 0 1"/></material>
     </visual>
     <collision>
       <origin xyz="0 0 0" rpy="0 0 0"/>
-      <geometry>
-        <cylinder radius="0.05" length="0.05"/>
-      </geometry>
+      <geometry><cylinder radius="0.05" length="0.05"/></geometry>
     </collision>
     <inertial>
       <mass value="0.1"/>
       <origin xyz="0 0 0" rpy="0 0 0"/>
-      <inertia ixx="0.0001" ixy="0.0" ixz="0.0"
-               iyy="0.0001" iyz="0.0"
-               izz="0.0001"/>
+      <inertia ixx="0.0001" ixy="0.0" ixz="0.0" iyy="0.0001" iyz="0.0" izz="0.0001"/>
     </inertial>
   </link>
   <joint name="lidar_joint" type="fixed">
-    <parent link="base_link"/>
+    <parent link="body"/>
     <child link="lidar_link"/>
     <origin xyz="0 0 0.1" rpy="0 0 0"/>
   </joint>
-  <!-- ============================================================ -->
-  <!-- IMU Link —— 物理实体                                          -->
-  <!-- ============================================================ -->
   <link name="imu_link">
     <inertial>
       <mass value="0.01"/>
       <origin xyz="0 0 0" rpy="0 0 0"/>
-      <inertia ixx="0.00001" ixy="0.0" ixz="0.0"
-               iyy="0.00001" iyz="0.0"
-               izz="0.00001"/>
+      <inertia ixx="0.00001" ixy="0.0" ixz="0.0" iyy="0.00001" iyz="0.0" izz="0.00001"/>
     </inertial>
   </link>
   <joint name="imu_joint" type="fixed">
-    <parent link="base_link"/>
+    <parent link="body"/>
     <child link="imu_link"/>
     <origin xyz="0 0 0.1" rpy="0 0 0"/>
   </joint>
   <!-- ============================================================ -->
-  <!-- 必须将 Ignition 传感器包裹在 gazebo 标签内，防止被 urdfdom 丢弃 -->
+  <!-- Ignition 传感器插件                                            -->
   <!-- ============================================================ -->
-  <!-- 1. Ignition GPU LiDAR 传感器 (16 线 3D) -->
-  <!-- 1. Mid-360 几何等效 CPU 激光雷达 (360° x 59°  hemispherical FOV) -->
   <gazebo reference="lidar_link">
-    <!-- 使用高度稳定的 CPU 射线追踪器，完全避免显卡驱动冲突 -->
-    <sensor type="lidar" name="lidar_sensor">
+    <sensor type="gpu_lidar" name="lidar_sensor">
       <pose>0 0 0.03 0 0 0</pose>
       <topic>/lidar/points</topic>
@@ -93,5 +95,5 @@
         <scan>
           <horizontal>
-            <samples>400</samples> <!-- 水平采样，RK3588 CPU 运行毫无压力 -->
+            <samples>400</samples>
             <resolution>1</resolution>
             <min_angle>-${M_PI}</min_angle>
@@ -99,20 +101,15 @@
           </horizontal>
           <vertical>
-            <samples>64</samples>  <!-- 64线高密度探测，1:1 还原 Mid-360 的立体扫描包络 -->
+            <samples>32</samples>
             <resolution>1</resolution>
-            <min_angle>-0.122173</min_angle> <!-- -7度 (向下) -->
-            <max_angle>0.907571</max_angle>  <!-- +52度 (向上) -->
+            <min_angle>-0.122173</min_angle>
+            <max_angle>0.907571</max_angle>
           </vertical>
         </scan>
         <range>
-          <min>0.1</min> <!-- 还原 Mid-360 0.1米极小盲区 -->
-          <max>40.0</max> <!-- 还原 Mid-360 40米最大测距 -->
+          <min>0.1</min>
+          <max>40.0</max>
           <resolution>0.001</resolution>
         </range>
-        <noise>
-          <type>gaussian</type>
-          <mean>0.0</mean>
-          <stddev>0.02</stddev> <!-- 注入高斯噪声，模拟真实的测量抖动 -->
-        </noise>
       </lidar>
       <always_on>1</always_on>
@@ -120,5 +117,4 @@
     </sensor>
   </gazebo>
-  <!-- 2. Ignition IMU 传感器 (200 Hz，恢复真实 6 轴噪声模型) -->
   <gazebo reference="imu_link">
     <sensor type="imu" name="imu_sensor">
@@ -142,3 +138,38 @@
     </sensor>
   </gazebo>
+  <!-- ============================================================ -->
+  <!-- ★ 核心修复：Ignition 标准多关节差速驱动系统 (4WD 四驱滑移转向)   -->
+  <!-- ============================================================ -->
+  <gazebo>
+    <plugin
+      filename="libignition-gazebo-diff-drive-system.so"
+      name="ignition::gazebo::systems::DiffDrive">
+      <!-- 绑定左侧前后两个轮子的关节 -->
+      <left_joint>left_front_wheel_joint</left_joint>
+      <left_joint>left_rear_wheel_joint</left_joint>
+      <!-- 绑定右侧前后两个轮子的关节 -->
+      <right_joint>right_front_wheel_joint</right_joint>
+      <right_joint>right_rear_wheel_joint</right_joint>
+      <wheel_separation>0.36</wheel_separation> <!-- 轮距 -->
+      <wheel_radius>0.08</wheel_radius>        <!-- 轮子半径 -->
+      <odom_publish_frequency>20</odom_publish_frequency> <!-- 里程计发布频率 -->
+      <!-- 速度命令与里程计话题 -->
+      <topic>/model/outdoor_bot/cmd_vel</topic>
+      <odom_topic>/odom</odom_topic>
+    </plugin>
+  </gazebo>
+  <!-- ============================================================ -->
+  <!-- ★ 修复：关节状态发布插件（让 RViz2 能渲染车轮转动）              -->
+  <!-- ============================================================ -->
+  <gazebo>
+    <plugin
+      filename="libignition-gazebo-joint-state-publisher-system.so"
+      name="ignition::gazebo::systems::JointStatePublisher">
+      <update_rate>30</update_rate>
+      <joint_name>left_front_wheel_joint</joint_name>
+      <joint_name>left_rear_wheel_joint</joint_name>
+      <joint_name>right_front_wheel_joint</joint_name>
+      <joint_name>right_rear_wheel_joint</joint_name>
+    </plugin>
+  </gazebo>
 </robot>
